File: Power_Solder/Power_Solder.kicad_sch (KiCad schematic)
At the start: 114 parts, among them IC1 MP1584EN, J1 HOTAIR HEAT, J2 HOTAIR SENSOR, J3 SOLDER HEAT, J4 SOLDER SENSOR, J5 220V IN, J6 24V IN, K1 FINDER-40.52, Q1 S8050, Q10 IRFR3708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

Commit message: Add files via upload
Parts:
- removed C20: 47uF, Capacitor_SMD:CP_Elec_5x5.4, symbol Device:C_Polarized_Small
- removed R48: 680k/1W, Resistor_SMD:R_1206_3216Metric, symbol Device:R_Small
- removed RV1, RV2: VDR, Varistor:RV_Disc_D7mm_W3.4mm_P5mm, symbol Device:Varistor
- added C20: 1uF, Capacitor_SMD:C_0603_1608Metric, symbol Device:C_Small
- added C23: 220uF, Capacitor_SMD:CP_Elec_6.3x7.7, symbol Device:C_Polarized_Small
- added C24, C25, C26, C27: 100nF, Capacitor_SMD:C_0603_1608Metric, symbol Device:C_Small
- added D16: SS34, Diode_SMD:D_SMA, symbol Diode:CDBA340-HF
- added J7: SOLDER SENSOR, XH_2.54mm_Conn:XH_3P_2.54mm_Vertical, symbol Connector:Conn_01x03_Male
Connections:
- net VIBRA SENSOR is gone; now on net SOLDER VIBRA: J4.2 (Pin_2)
- net +12V: now also C23.1
- net +24V: now also D16.2 (A); no longer IC1.7 (VIN), R3.1
- net +3.3V: now also C27.2
- net +5V: now also C24.2, C25.2, C26.2, J7.1 (Pin_1)
- net AC1: now also U5.3 (IP-), U5.4 (IP-); no longer U5.1 (IP+), U5.2 (IP+)
- net AC1i: now also K1.11, U5.1 (IP+), U5.2 (IP+); no longer K1.24, U5.3 (IP-), U5.4 (IP-)
- net AC2: now also J1.1 (Pin_1), K1.21; no longer J1.2 (Pin_2), K1.14
- net AC_L: now also J5.1 (Pin_1); no longer J5.3 (Pin_3)
- net AC_N: now also K1.14; no longer K1.21
- net Earth_Protective: now also J1.3 (Pin_3), J3.3 (Pin_3), J5.3 (Pin_3); no longer J1.1 (Pin_1), J3.1 (Pin_1), J5.1 (Pin_1)
- net GND: now also C20.2, C23.2, C24.1, C25.1, C26.1, C27.1, J7.2 (Pin_2)
- net HOTAIR HEAT: now also J1.2 (Pin_2); no longer J1.3 (Pin_3)
- net SOLDER HEAT: now also J3.1 (Pin_1); no longer J3.3 (Pin_3)
- net SPEAKER: now also J7.3 (Pin_3)
- net at C17.1, F1.2: now also K1.24; no longer K1.11
- new net: C20.1, D16.1 (K), IC1.7 (VIN), R3.1
Other:
- moved on the sheet: C17, F1, J1, J3, J5
